Commit message: Switched to position control. Added python script to publish trajectories.

File: kr270_description/urdf/kr270.urdf (robot description, URDF)
Before this commit: robot kr270, 7 links, 6 joints
Joints:
- joint joint_a1: limit lower=-3 upper=3 effort=10000.0 velocity=100.0 -> lower=-3.2289 upper=3.2289 effort=10000.0 velocity=100.0
- joint joint_a4: limit lower=-3 upper=3 effort=10000.0 velocity=100.0 -> lower=-6.109 upper=6.109 effort=10000.0 velocity=100.0

Commit message: Adds high res meshes.

File: kr270_description/urdf/kr270.urdf (robot description, URDF)
Before this commit: robot kr270, 7 links, 6 joints
Links:
- link a1: geometry collision box size=.5 .25 .3; collision cylinder length=.3 radius=.2
- link a2: geometry collision box size=.3 .3 1.3; collision cylinder length=.2 radius=.2
- link a3: geometry collision box size=.6 .4 .15; collision cylinder length=1.2 radius=0.15
- link a4: geometry collision cylinder length=0.5 radius=0.1; visual cylinder length=0.5 radius=0.1
- link a5: geometry collision cylinder length=0.08 radius=0.1; collision cylinder length=0.3 radius=0.125
- link socket: geometry collision box size=.3 .3 .3; collision box size=.7 .7 .2

Commit message: Fixed high-res mesh for KR270. Added lighting to world file.

File: kr270_description/urdf/kr270.urdf (robot description, URDF)
Before this commit: robot kr270, 7 links, 6 joints
Links:
- link a1: geometry collision box size=.5 .25 .3; collision cylinder length=.3 radius=.2
- link a2: geometry collision box size=.3 .3 1.3; collision cylinder length=.2 radius=.2
- link a3: geometry collision box size=.65 .4 .15; collision cylinder length=1.3 radius=0.15
- link a4: geometry collision cylinder length=0.4 radius=0.1; visual mesh filename=package://kr270_description/meshes/A4.dae scale=0.025 0.025 0.025
- link a5: geometry collision cylinder length=0.08 radius=0.1; collision cylinder length=0.3 radius=0.125
- link socket: geometry collision box size=.3 .3 .3; collision box size=.7 .7 .2
Joints:
- joint joint_a4: origin xyz=-1 0 0 rpy=0 0 0 -> xyz=-1 0 -0.045 rpy=0 0 0
- joint joint_a5: limit lower=-3.709 upper=0.567 effort=10000.0 velocity=100.0 -> lower=-2.138 upper=2.138 effort=10000.0 velocity=100.0
